File: separation/v2_hackspace.brd (EAGLE design)
At the start: 40.6 x 25.4 mm, 10 parts

Commit message: complete hackspace pcb
Parts:
- moved C2 32.6 mm to (17.4, 13.6), turned to 270 degrees
- moved C1 29.5 mm to (17.3, 19.9), turned to 270 degrees
- moved R2 27.2 mm to (-12.2, 19.3), turned to 90 degrees
- moved R1 18.3 mm to (-15.4, 19.3), turned to 90 degrees
- moved LDO 5.47 mm to (13.0, 14.6), turned to 90 degrees
- moved LOUD 2.01 mm to (14.5, 8.00), turned to 270 degrees
- moved SERCON 0.63 mm to (-15.0, 4.19)
Routing:
- net VSENSE: track 36.5 -> 8.83 mm
- net VCC: track 34.3 -> 10.4 mm
- net GND: track 0.00 -> 11.2 mm
- net VBAT: track 62.3 -> 68.0 mm
- net BUZZ: track 9.01 -> 7.83 mm
- net SERVO: track 15.4 -> 14.8 mm
